File: wave_light.kicad_pcb (KiCad board)
At the start: 2 copper layers, 0 parts

Commit message: Redesign with rectangular layout
Parts:
- added C1: CP1, Capacitor_SMD:C_1206_3216Metric_Pad1.42x1.75mm_HandSolder, F.Cu at (72.2, 76.5)
- added J1: Conn_01x02_Male, Connector_JST:JST_XH_B2B-XH-A_1x02_P2.50mm_Vertical, F.Cu at (70.9, 71.1)
- added J2: Conn_01x02_Male, Connector_JST:JST_XH_B2B-XH-A_1x02_P2.50mm_Vertical, F.Cu at (81.0, 69.6)
- added J3: Conn_01x02_Male, Connector_JST:JST_XH_B2B-XH-A_1x02_P2.50mm_Vertical, F.Cu at (89.4, 69.6)
- added J4: Conn_01x02_Male, Connector_JST:JST_XH_B2B-XH-A_1x02_P2.50mm_Vertical, F.Cu at (97.8, 69.6)
- added J5: Conn_01x02_Male, Connector_JST:JST_XH_B2B-XH-A_1x02_P2.50mm_Vertical, F.Cu at (106.2, 69.6)
- added J6: Conn_01x02_Male, Connector_JST:JST_XH_B2B-XH-A_1x02_P2.50mm_Vertical, F.Cu at (114.6, 69.6)
- added J7: Conn_01x02_Male, Connector_JST:JST_XH_B2B-XH-A_1x02_P2.50mm_Vertical, F.Cu at (122.9, 69.6)
- added J8: Conn_01x02_Male, Connector_JST:JST_XH_B2B-XH-A_1x02_P2.50mm_Vertical, F.Cu at (131.3, 69.6)
- added J9: Conn_01x02_Male, Connector_JST:JST_XH_B2B-XH-A_1x02_P2.50mm_Vertical, F.Cu at (139.7, 69.6)
- added R1: R_US, Resistor_SMD:R_1206_3216Metric_Pad1.42x1.75mm_HandSolder, F.Cu at (80.5, 76.7)
- added R2: R_US, Resistor_SMD:R_1206_3216Metric_Pad1.42x1.75mm_HandSolder, F.Cu at (88.9, 76.7)
- added R3: R_US, Resistor_SMD:R_1206_3216Metric_Pad1.42x1.75mm_HandSolder, F.Cu at (97.2, 76.7)
- added R4: R_US, Resistor_SMD:R_1206_3216Metric_Pad1.42x1.75mm_HandSolder, F.Cu at (105.6, 76.7)
- added R5: R_US, Resistor_SMD:R_1206_3216Metric_Pad1.42x1.75mm_HandSolder, F.Cu at (114.0, 76.7)
- added R6: R_US, Resistor_SMD:R_1206_3216Metric_Pad1.42x1.75mm_HandSolder, F.Cu at (122.4, 76.7)
- added R7: R_US, Resistor_SMD:R_1206_3216Metric_Pad1.42x1.75mm_HandSolder, F.Cu at (130.8, 76.7)
- added R8: R_US, Resistor_SMD:R_1206_3216Metric_Pad1.42x1.75mm_HandSolder, F.Cu at (138.9, 76.7)
Routing:
- net Net-(J7-Pad2): track 0.00 -> 5.00 mm
- net Net-(J6-Pad2): track 0.00 -> 5.00 mm
- net Net-(J5-Pad2): track 0.00 -> 5.00 mm
- net Net-(J4-Pad2): track 0.00 -> 5.00 mm
- net Net-(J3-Pad2): track 0.00 -> 5.00 mm
- net Net-(J2-Pad2): track 0.00 -> 5.00 mm
- net Net-(J8-Pad2): track 0.00 -> 5.00 mm
- net Net-(J9-Pad2): track 0.00 -> 4.86 mm
- net GND: track 0.00 -> 1.85 mm, vias 0 -> 1
- added copper zone on F.Cu, net +5V
- added copper zone on B.Cu, net GND
Other:
- board outline added: 86.4 x 14 mm
- board text added: "-PWR IN+"
